Commit message: zarm-sim: the 310 mm stroke fits Hitbot's stock column; frame the whole arm
User feedback: "The vertical range of the robot sim doesn't seem to cover the full
range of the cad file". The old mesh stretch grew the CAD column by 103 mm over
130-470 mm (to a 696 mm column from the spec's 596 for a 210 mm stroke), so the J1
housing never reached the top of the column's slots.

Measured in the STEP (down the middle of the two front slots): the slots are open
from 172 mm (above the electronics bay's bracket) to the cap at 578 mm; the J1
housing spans 134.9 to 195.9 mm above the flange face; the column is 593 mm (596
with the drawing's 3 mm lid, the spec's height). The drawing's two positions are
240 mm apart (flange faces 63.9 and 304.0 mm, kept as cad_stroke_mm, information).

Coordinator decision: the 310 mm stroke fits the stock column. The flange face
runs 64 -> 374 mm as before, and the J1 housing sweeps 198.9 -> 569.9 mm, leaving
26.9 mm of slot below and 8.1 mm under the cap. The column grows only for a stroke
over 318.1 mm, by exactly the shortfall, stretching the plain middle the housing
sweeps over the drawn travel; the slot's end and the cap move up unchanged.

- dimensions.py: cad_column_height_mm, cad_lid_height_mm, cad_slot_bottom_mm,
  cad_stroke_mm and housing_bottom_above_flange_mm (STEP: 3 mm above the J1 arm)
  with sources; column_growth_mm, travel_zone_mm(), slot_clearances_mm().
- URDF/MJCF regenerated: the column is 593 mm to its cap (was 696).
- fetch_cad_meshes.py measures the slot and the housing in the STEP, checks
  them, and grows the column only when needed (not for 310 mm).
- The view frames the whole arm, base plate to column top, at the canvas's
  aspect (a 500 x 1090 side panel too), refitting on resize until the camera is
  moved; Reset view refits. The J3 rail gets an end stop at each end of travel.
- Tests: the housing's sweep within the slot with those clearances, in the URDF
  and in the CAD meshes; every stroke option; the growth for 410/510 mm.

Co-authored-by: Copilot App <223556219+Copilot@users.noreply.github.com>

File: zarm-sim/models/zarm_2442.urdf (robot description, URDF)
Before this commit: robot zarm_2442, 7 links, 6 joints
Links:
- link base_link: geometry collision box size=0.128 0.148 0.015; collision box size=0.128 0.148 0.568
- link carriage: geometry collision box size=0.069 0.1 0.061; collision cylinder length=0.061 radius=0.05
